File: _saved_ESP_LOGGER.sch (KiCad schematic (older format))
At the start: 25 parts, among them SW1 SW_Push, SW2 SW_Push, U1 AZ1086_SOT223

Commit message: schematic
Parts:
- MPU1: footprint Pin_Headers:Pin_Header_Straight_2x02_Pitch2.54mm -> Pin_Headers:Pin_Header_Straight_1x04_Pitch2.54mm
Changed lines of the file:
@@
 F 0 "MPU1" H 2894 1425 50  0000 C CNN
 F 1 "Conn_01x04_Female" H 2894 1516 50  0000 C CNN
-F 2 "Pin_Headers:Pin_Header_Straight_2x02_Pitch2.54mm" H 3000 1850 50  0001 C CNN
+F 2 "Pin_Headers:Pin_Header_Straight_1x04_Pitch2.54mm" H 3000 1850 50  0001 C CNN
 F 3 "~" H 3000 1850 50  0001 C CNN
 	1    3000 1850
