File: ESP_LOGGER.sch (KiCad schematic (older format))
At the start: 25 parts, among them SW1 SW_Push, SW2 SW_Push, U1 AZ1086_SOT223

Commit message: pcb F.Cu
Parts:
- removed BATTERY1: Conn_01x02_Female, Connectors_Molex:Molex_PicoBlade_53047-0210_02x1.25mm_Straight, symbol Connector:Conn_01x02_Female
- removed ESP_I2C1, ESP_PWR1: Conn_01x02_Female, Pin_Headers:Pin_Header_Straight_1x02_Pitch2.54mm, symbol Connector:Conn_01x02_Female
- removed ESP_LED1: Conn_01x01_Female, Pin_Headers:Pin_Header_Straight_1x01_Pitch2.54mm, symbol Connector:Conn_01x01_Female
- removed ESP_SD1: Conn_01x05_Female, Pin_Headers:Pin_Header_Straight_1x05_Pitch2.54mm, symbol Connector:Conn_01x05_Female
- removed FTDI1: Conn_01x05_Male, Pin_Headers:Pin_Header_Straight_1x05_Pitch2.54mm, symbol Connector:Conn_01x05_Male
- added ESP_COM1: Conn_01x08_Female, Connector_PinSocket_2.54mm:PinSocket_1x08_P2.54mm_Vertical, symbol Connector:Conn_01x08_Female
- added ESP_VDD1: Conn_01x02_Female, Connector_PinSocket_2.54mm:PinSocket_1x02_P2.54mm_Vertical, symbol Connector:Conn_01x02_Female
- added JBATT1: Conn_01x02_Female, Connector_Molex:Molex_PicoBlade_53047-0410_1x02_P1.25mm_Vertical, symbol Connector:Conn_01x02_Female
- added JFTDI1: Conn_01x05_Female, Connector_PinSocket_2.54mm:PinSocket_1x05_P2.54mm_Vertical, symbol Connector:Conn_01x05_Female
- added TP1, TP2, TP3, TP4, TP5, TP7: TestPoint, TestPoint:TestPoint_Loop_D2.54mm_Drill1.5mm_Beaded, symbol Connector:TestPoint
- C1: value 10uF -> 100u; footprint Capacitors_SMD:C_0805_HandSoldering -> Capacitor_SMD:C_0805_2012Metric_Pad1.15x1.40mm_HandSolder
- C2: value 0.1uF -> 1u; footprint Capacitors_SMD:C_0805_HandSoldering -> Capacitor_SMD:C_0805_2012Metric_Pad1.15x1.40mm_HandSolder
- C3, C4: value 1nF -> 1n; footprint Capacitors_SMD:C_0805_HandSoldering -> Capacitor_SMD:C_0805_2012Metric_Pad1.15x1.40mm_HandSolder
- D1: footprint Diodes_ThroughHole:D_5W_P10.16mm_Horizontal -> Diode_THT:D_A-405_P7.62mm_Horizontal
- D2: footprint Diodes_ThroughHole:D_T-1_P2.54mm_Vertical_AnodeUp -> LED_THT:LED_D5.0mm_Clear
- ESP_SWT1, ESP_UART1: footprint Pin_Headers:Pin_Header_Straight_1x02_Pitch2.54mm -> Connector_PinSocket_2.54mm:PinSocket_1x02_P2.54mm_Vertical
- MICROSD1: footprint Pin_Headers:Pin_Header_Straight_1x08_Pitch2.54mm -> Connector_PinSocket_2.54mm:PinSocket_1x08_P2.54mm_Vertical
- MPU1: footprint Pin_Headers:Pin_Header_Straight_2x02_Pitch2.54mm -> Connector_PinSocket_2.54mm:PinSocket_1x04_P2.54mm_Vertical
- R1, R2, R3: value 10k -> R; footprint Resistors_ThroughHole:R_Axial_DIN0207_L6.3mm_D2.5mm_P10.16mm_Horizontal -> Resistor_THT:R_Axial_DIN0207_L6.3mm_D2.5mm_P10.16mm_Horizontal
- R4, R5, R6: footprint Resistors_ThroughHole:R_Axial_DIN0207_L6.3mm_D2.5mm_P10.16mm_Horizontal -> Resistor_THT:R_Axial_DIN0207_L6.3mm_D2.5mm_P10.16mm_Horizontal
- SW1, SW2: footprint Buttons_Switches_SMD:SW_SPST_EVQPE1 -> Button_Switch_THT:SW_PUSH_6mm
- U1: footprint TO_SOT_Packages_SMD:SOT-223-3_TabPin2 -> Package_TO_SOT_SMD:SOT-223
Connections:
- net labels added: J_CD, J_CLK
- net labels removed: VCC
- wire segments 68 -> 82

Commit message: bugfix
Parts:
- R2, R3: value R -> 10k
Connections:
- wire segments 82 -> 85
Changed lines of the file:
@@
 Text GLabel 1350 4650 0    50   Input ~ 0
 GND
-Text GLabel 2850 4350 0    50   Input ~ 0
+Text GLabel 2850 4700 0    50   Input ~ 0
 BOOT
 Wire Wire Line
@@
 	3500 5650 3350 5650
 Wire Wire Line
-	3350 5650 3350 5300
+	3350 5650 3350 5500
 Wire Wire Line
 	3300 5300 3350 5300
 Connection ~ 3350 5300
-Text GLabel 2850 5300 0    50   Input ~ 0
+Text GLabel 2800 5500 0    50   Input ~ 0
 EN
 Text GLabel 1350 5250 0    50   Input ~ 0
@@
 P 3150 4350
 F 0 "R2" V 2943 4350 50  0000 C CNN
-F 1 "R" V 3034 4350 50  0000 C CNN
+F 1 "10k" V 3034 4350 50  0000 C CNN
 F 2 "Resistor_THT:R_Axial_DIN0207_L6.3mm_D2.5mm_P10.16mm_Horizontal" V 3080 4350 50  0001 C CNN
 F 3 "~" H 3150 4350 50  0001 C CNN
@@
 P 3150 5300
 F 0 "R3" V 2943 5300 50  0000 C CNN
-F 1 "R" V 3034 5300 50  0000 C CNN
+F 1 "10k" V 3034 5300 50  0000 C CNN
 F 2 "Resistor_THT:R_Axial_DIN0207_L6.3mm_D2.5mm_P10.16mm_Horizontal" V 3080 5300 50  0001 C CNN
 F 3 "~" H 3150 5300 50  0001 C CNN
@@
 	0    -1   -1   0
 $EndComp
+Text GLabel 2850 5300 0    50   Input ~ 0
+3.3V
+Wire Wire Line
+	2800 5500 3350 5500
+Connection ~ 3350 5500
+Wire Wire Line
+	3350 5500 3350 5300
+Text GLabel 2850 4350 0    50   Input ~ 0
+3.3V
+Wire Wire Line
+	2850 4700 3350 4700
+Connection ~ 3350 4700
 $EndSCHEMATC

Commit message: improvement in the size and usability
Parts:
- removed D1: DIODE, Diode_THT:D_A-405_P7.62mm_Horizontal, symbol pspice:DIODE
- removed R5, R6: 10k, Resistor_THT:R_Axial_DIN0207_L6.3mm_D2.5mm_P10.16mm_Horizontal, symbol Device:R
- removed TP1, TP2, TP3, TP4, TP5, TP7: TestPoint, TestPoint:TestPoint_Loop_D2.54mm_Drill1.5mm_Beaded, symbol Connector:TestPoint
Connections:
- net labels added: CS, DI, SCK
- net labels removed: CLK, CMD, D3, J_CD, J_CLK, PC_5V, S_SCL, S_SDA
- wire segments 85 -> 71
- no-connect marks 2 -> 3
Changed lines of the file:
@@
 D0
 Text GLabel 2050 2300 2    50   Input ~ 0
-CLK
+SCK
 Text GLabel 2050 2500 2    50   Input ~ 0
-CMD
+DI
 Text GLabel 2050 2400 2    50   Input ~ 0
-D3
+CS
 Text GLabel 2050 1650 2    50   Input ~ 0
 GND
@@
 GND
 Text GLabel 3400 1850 2    50   Input ~ 0
-S_SCL
+SCL
 Text GLabel 3400 1950 2    50   Input ~ 0
-S_SDA
+SDA
 Wire Wire Line
 	3200 1650 3400 1650
@@
 	3200 1950 3400 1950
 Text GLabel 3400 2350 2    50   Input ~ 0
-D3
+CS
 Text GLabel 3400 2450 2    50   Input ~ 0
-CMD
+DI
 Text GLabel 3400 2550 2    50   Input ~ 0
 3.3V
-Text GLabel 3400 2650 2    50   Input ~ 0
-J_CLK
 Text GLabel 3400 2750 2    50   Input ~ 0
 GND
@@
 NoConn ~ 3200 2950
 Text GLabel 3400 3050 2    50   Input ~ 0
-J_CD
+CD
 Wire Wire Line
 	3200 3050 3400 3050
@@
 Text GLabel 4400 1650 2    50   Input ~ 0
 PC_GND
-Text GLabel 4400 1850 2    50   Input ~ 0
-PC_5V
 Text GLabel 4400 1950 2    50   Input ~ 0
 PC_TX
@@
 Wire Wire Line
 	5100 1650 5400 1650
-Text GLabel 4200 2400 0    50   Input ~ 0
-PC_5V
-Text GLabel 4200 2500 0    50   Input ~ 0
-PC_GND
 Text GLabel 4200 2850 0    50   Input ~ 0
 BATT
 Text GLabel 4200 2950 0    50   Input ~ 0
 BATT_GND
-Wire Wire Line
-	4200 2500 4800 2500
-Wire Wire Line
-	4200 2950 4800 2950
-Connection ~ 4800 2950
-Text GLabel 5250 2400 2    50   Input ~ 0
+Text GLabel 5300 2850 2    50   Input ~ 0
 POWER
 Text GLabel 5300 2950 2    50   Input ~ 0
@@
 Text GLabel 7000 2300 3    50   Input ~ 0
 3.3V
-Wire Wire Line
-	5000 2850 4750 2850
-Wire Wire Line
-	5000 2400 5000 2850
-Connection ~ 5000 2400
-Wire Wire Line
-	4800 2500 4800 2950
 Wire Wire Line
 	7700 1600 7900 1600
@@
 Wire Wire Line
 	1400 1650 2050 1650
-Text GLabel 5100 4300 0    50   Input ~ 0
-SCL
-Text GLabel 5100 4650 0    50   Input ~ 0
-SDA
-Text GLabel 5900 4650 2    50   Input ~ 0
-S_SCL
-Text GLabel 5900 4300 2    50   Input ~ 0
-S_SDA
-Wire Wire Line
-	5100 4300 5350 4300
-Wire Wire Line
-	5650 4300 5900 4300
-Wire Wire Line
-	5100 4650 5350 4650
-Wire Wire Line
-	5650 4650 5900 4650
 Wire Wire Line
 	3900 4350 4150 4350
@@
 Wire Wire Line
 	3350 5300 3450 5300
-Wire Wire Line
-	5000 2400 5250 2400
 $Comp
 L Connector:Conn_01x08_Female ESP_COM1
@@
 	-1   0    0    1
 $EndComp
-Wire Wire Line
-	4200 2400 5000 2400
-Wire Wire Line
-	4200 2850 4350 2850
 Wire Wire Line
 	1350 4350 1600 4350
@@
 	1    0    0    -1
 $EndComp
-Wire Wire Line
-	4800 2950 5300 2950
-$Comp
-L pspice:DIODE D1
-U 1 1 5BC93915
-P 4550 2850
-F 0 "D1" H 4550 3115 50  0000 C CNN
-F 1 "DIODE" H 4550 3024 50  0000 C CNN
-F 2 "Diode_THT:D_A-405_P7.62mm_Horizontal" H 4550 2850 50  0001 C CNN
-F 3 "~" H 4550 2850 50  0001 C CNN
-	1    4550 2850
-	1    0    0    -1
-$EndComp
 $Comp
 L Device:R R4
@@
 	1    5250 3400
 	-1   0    0    1
-$EndComp
-$Comp
-L Device:R R5
-U 1 1 5BC93B14
-P 5500 4300
-F 0 "R5" V 5293 4300 50  0000 C CNN
-F 1 "10k" V 5384 4300 50  0000 C CNN
-F 2 "Resistor_THT:R_Axial_DIN0207_L6.3mm_D2.5mm_P10.16mm_Horizontal" V 5430 4300 50  0001 C CNN
-F 3 "~" H 5500 4300 50  0001 C CNN
-	1    5500 4300
-	0    1    1    0
-$EndComp
-$Comp
-L Device:R R6
-U 1 1 5BC93B77
-P 5500 4650
-F 0 "R6" V 5293 4650 50  0000 C CNN
-F 1 "10k" V 5384 4650 50  0000 C CNN
-F 2 "Resistor_THT:R_Axial_DIN0207_L6.3mm_D2.5mm_P10.16mm_Horizontal" V 5430 4650 50  0001 C CNN
-F 3 "~" H 5500 4650 50  0001 C CNN
-	1    5500 4650
-	0    1    1    0
 $EndComp
 $Comp
@@
 	-1   0    0    1
 $EndComp
-Text GLabel 6500 2900 0    50   Input ~ 0
-CD
-Text GLabel 6500 3200 0    50   Input ~ 0
-CLK
-Text GLabel 7500 3200 2    50   Input ~ 0
-J_CLK
-Text GLabel 7500 2900 2    50   Input ~ 0
-J_CD
-Wire Wire Line
-	6500 2900 6700 2900
-Wire Wire Line
-	7300 2900 7500 2900
-Wire Wire Line
-	7500 3200 7300 3200
-Wire Wire Line
-	6500 3200 6700 3200
-$Comp
-L Connector:TestPoint TP1
-U 1 1 5BCA46F6
-P 6700 2900
-F 0 "TP1" V 6654 3088 50  0000 L CNN
-F 1 "TestPoint" V 6745 3088 50  0000 L CNN
-F 2 "TestPoint:TestPoint_Loop_D2.54mm_Drill1.5mm_Beaded" H 6900 2900 50  0001 C CNN
-F 3 "~" H 6900 2900 50  0001 C CNN
-	1    6700 2900
-	0    1    1    0
-$EndComp
-$Comp
-L Connector:TestPoint TP2
-U 1 1 5BCA480A
-P 6700 3200
-F 0 "TP2" V 6654 3388 50  0000 L CNN
-F 1 "TestPoint" V 6745 3388 50  0000 L CNN
-F 2 "TestPoint:TestPoint_Loop_D2.54mm_Drill1.5mm_Beaded" H 6900 3200 50  0001 C CNN
-F 3 "~" H 6900 3200 50  0001 C CNN
-	1    6700 3200
-	0    1    1    0
-$EndComp
-$Comp
-L Connector:TestPoint TP3
-U 1 1 5BCA4854
-P 7300 2900
-F 0 "TP3" V 7495 2974 50  0000 C CNN
-F 1 "TestPoint" V 7404 2974 50  0000 C CNN
-F 2 "TestPoint:TestPoint_Loop_D2.54mm_Drill1.5mm_Beaded" H 7500 2900 50  0001 C CNN
-F 3 "~" H 7500 2900 50  0001 C CNN
-	1    7300 2900
-	0    -1   -1   0
-$EndComp
-$Comp
-L Connector:TestPoint TP4
-U 1 1 5BCA48F0
-P 7300 3200
-F 0 "TP4" V 7495 3274 50  0000 C CNN
-F 1 "TestPoint" V 7404 3274 50  0000 C CNN
-F 2 "TestPoint:TestPoint_Loop_D2.54mm_Drill1.5mm_Beaded" H 7500 3200 50  0001 C CNN
-F 3 "~" H 7500 3200 50  0001 C CNN
-	1    7300 3200
-	0    -1   -1   0
-$EndComp
-Text GLabel 6500 3600 0    50   Input ~ 0
-GND
-Text GLabel 7500 3600 2    50   Input ~ 0
-GND
-Wire Wire Line
-	7500 3600 7300 3600
-Wire Wire Line
-	6500 3600 6700 3600
-$Comp
-L Connector:TestPoint TP5
-U 1 1 5BCAFF4C
-P 6700 3600
-F 0 "TP5" V 6654 3788 50  0000 L CNN
-F 1 "TestPoint" V 6745 3788 50  0000 L CNN
-F 2 "TestPoint:TestPoint_Loop_D2.54mm_Drill1.5mm_Beaded" H 6900 3600 50  0001 C CNN
-F 3 "~" H 6900 3600 50  0001 C CNN
-	1    6700 3600
-	0    1    1    0
-$EndComp
-$Comp
-L Connector:TestPoint TP7
-U 1 1 5BCAFF53
-P 7300 3600
-F 0 "TP7" V 7495 3674 50  0000 C CNN
-F 1 "TestPoint" V 7404 3674 50  0000 C CNN
-F 2 "TestPoint:TestPoint_Loop_D2.54mm_Drill1.5mm_Beaded" H 7500 3600 50  0001 C CNN
-F 3 "~" H 7500 3600 50  0001 C CNN
-	1    7300 3600
-	0    -1   -1   0
-$EndComp
 Text GLabel 2850 5300 0    50   Input ~ 0
 3.3V
@@
 	2850 4700 3350 4700
 Connection ~ 3350 4700
+Text GLabel 3400 2650 2    50   Input ~ 0
+SCK
+Wire Wire Line
+	4200 2950 4800 2950
+Wire Wire Line
+	4200 2850 5300 2850
+NoConn ~ 4400 1850
+Text GLabel 5300 3050 2    50   Input ~ 0
+PC_GND
+Wire Wire Line
+	5300 3050 4800 3050
+Wire Wire Line
+	4800 3050 4800 2950
+Connection ~ 4800 2950
+Wire Wire Line
+	4800 2950 5300 2950
 $EndSCHEMATC
